Commit message: 230324

File: patrol_scout_mini_dw/patrol_scout_mini/scout_description/urdf/mini.xacro (robot description, xacro)
@@ -64,5 +64,5 @@
     </link>
     <joint name="inertial_joint" type="fixed">
-        <origin xyz="0 0 0" rpy="0 0 0" />
+        <origin xyz="3 3 0" rpy="0 0 0" />
         <parent link="base_link" />
         <child link="inertial_link" />
